File: projects/starter.brd (EAGLE design)
At the start: 50.8 x 50.9 mm, 32 parts, among them CN1 MiniB USB, IC1 ATMEGA32U4-AU, X3 16MHz

Commit message: prep for feb 5th class
Parts:
- removed U$3, U$5, U$7, U$8: DOTSTAR, codenext2020:SK9822
- moved U$6 5.00 mm to (16.6, 27.3)
- moved BOOT 5.00 mm to (37.9, 24.8)
- moved C1 5.00 mm to (11.8, 16.2)
- moved C2 5.00 mm to (40.5, 16.5)
- moved C3 5.00 mm to (40.5, 20.1)
- moved C4 5.00 mm to (12.2, 27.8)
- moved C5 5.00 mm to (12.7, 25.8)
- moved C6 5.00 mm to (32.2, 17.3)
- moved C7 5.00 mm to (31.1, 28.0)
- moved CN1 5.00 mm to (4.41, 22.0)
- moved IC1 5.00 mm to (24.0, 21.7)
- moved ISP6 5.00 mm to (47.7, 22.0)
- moved JP1 5.00 mm to (24.7, 11.8)
- moved JP5 5.00 mm to (24.7, 32.2)
- moved L 5.00 mm to (3.39, 15.1)
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Connections:
- removed net N$11: U$3.SDO, U$5.SDI
- removed net N$12: U$3.CKO, U$5.CKI
- removed net N$13: U$5.SDO, U$7.SDI
- removed net N$14: U$5.CKO, U$7.CKI
- removed net N$15: U$7.SDO, U$8.SDI
- removed net N$16: U$7.CKO, U$8.CKI
- net +5V: no longer U$3.VCC, U$5.VCC, U$7.VCC, U$8.VCC
- net GND: no longer U$3.GND, U$5.GND, U$7.GND, U$8.GND
- net MOSI: no longer U$3.SDI
- net SCK: no longer U$3.CKI
Routing:
- net +5V: track 94.9 -> 32.1 mm, vias 2 -> 1
- net GND: track 43.6 -> 1.14 mm, vias 12 -> 8
- net SCK: track 80.5 -> 65.2 mm
- net MOSI: track 67.3 -> 53.0 mm
- net N$14: track 4.10 -> 0.00 mm
- net N$13: track 4.10 -> 0.00 mm
- net N$12: track 4.10 -> 0.00 mm
- net N$11: track 4.10 -> 0.00 mm
- net N$16: track 4.10 -> 0.00 mm
- net N$15: track 4.10 -> 0.00 mm
- net PF0: track 14.5 -> 13.1 mm
Other:
- board size 50.8 x 50.9 mm -> 50.8 x 34.9 mm
