File: projects/starter.sch (EAGLE design)
At the start: 31 parts, among them CN1 MiniB USB, IC1 ATMEGA32U4-AU, X3 16MHz

Commit message: prep for feb 5th class
Parts:
- removed U$3, U$5, U$7, U$8: DOTSTAR, codenext2020:DOTSTAR
Connections:
- removed net N$11: U$3.DO, U$5.DI
- removed net N$12: U$3.CO, U$5.CI
- removed net N$13: U$5.DO, U$7.DI
- removed net N$14: U$5.CO, U$7.CI
- removed net N$15: U$7.DO, U$8.DI
- removed net N$16: U$7.CO, U$8.CI
- net +5V: no longer U$3.VCC, U$5.VCC, U$7.VCC, U$8.VCC
- net GND: no longer U$3.GND, U$5.GND, U$7.GND, U$8.GND
- net MOSI: no longer U$3.DI
- net SCK: no longer U$3.CI
