File: projects/atmega32u4bb.sch (EAGLE design)
At the start: 31 parts, among them CN1 MiniB USB, IC1 ATMEGA32U4-AU, X3 16MHz

Commit message: Add 2020 (2mm by 2mm) footprint for dotstar, updated example to use that footprint
Parts:
- U$3, U$5, U$7, U$8: value DOTSTAR -> DOTSTAR2020; device codenext2020:DOTSTAR -> codenext2020:DOTSTAR2020
Changed lines of the file:
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@@
 <part name="U$6" library="adafruit" deviceset="FIDUCIAL" device=""/>
 <part name="FRAME1" library="frames" deviceset="FRAME_A_L" device=""/>
-<part name="U$3" library="codenext2020" deviceset="DOTSTAR" device=""/>
-<part name="U$5" library="codenext2020" deviceset="DOTSTAR" device=""/>
-<part name="U$7" library="codenext2020" deviceset="DOTSTAR" device=""/>
-<part name="U$8" library="codenext2020" deviceset="DOTSTAR" device=""/>
+<part name="U$3" library="codenext2020" deviceset="DOTSTAR" device="2020"/>
+<part name="U$5" library="codenext2020" deviceset="DOTSTAR" device="2020"/>
+<part name="U$7" library="codenext2020" deviceset="DOTSTAR" device="2020"/>
+<part name="U$8" library="codenext2020" deviceset="DOTSTAR" device="2020"/>
 <part name="GND11" library="supply1" deviceset="GND" device=""/>
 <part name="V5" library="supply2" deviceset="+5V" device=""/>
@@
 <wire x1="102" y1="48" x2="102" y2="44" width="0.1524" layer="91"/>
 <pinref part="GND11" gate="1" pin="GND"/>
-<wire x1="102" y1="44" x2="104.08" y2="44" width="0.1524" layer="91"/>
-<wire x1="104.08" y1="44" x2="104.08" y2="41.4" width="0.1524" layer="91"/>
+<wire x1="104" y1="44" x2="104.08" y2="41.4" width="0.1524" layer="91"/>
+<wire x1="102" y1="44" x2="104" y2="44" width="0.1524" layer="91"/>
 <pinref part="U$5" gate="G$1" pin="GND"/>
-<wire x1="104.08" y1="44" x2="135" y2="44" width="0.1524" layer="91"/>
 <wire x1="135" y1="44" x2="135" y2="48" width="0.1524" layer="91"/>
 <pinref part="U$7" gate="G$1" pin="GND"/>
 <wire x1="135" y1="44" x2="166" y2="44" width="0.1524" layer="91"/>
 <wire x1="166" y1="44" x2="166" y2="48" width="0.1524" layer="91"/>
-<junction x="135" y="44"/>
 <wire x1="166" y1="44" x2="193" y2="44" width="0.1524" layer="91"/>
 <wire x1="193" y1="44" x2="193" y2="67" width="0.1524" layer="91"/>
@@
 <pinref part="U$8" gate="G$1" pin="GND"/>
 <wire x1="193" y1="67" x2="188" y2="67" width="0.1524" layer="91"/>
+<wire x1="104" y1="44" x2="135" y2="44" width="0.1524" layer="91"/>
+<junction x="104" y="44"/>
+<junction x="135" y="44"/>
 </segment>
 </net>
